Commit message: get all param in one file

File: cartographer_ros/urdf/m6_cky.urdf (robot description, URDF)
Before this commit: robot cartographer_backpack_3d, 5 links, 4 joints
Joints:
- joint imu_link_joint: origin xyz=0 0 0 rpy=3.14159 0.0 1.57 -> xyz=0.0 0.0 0.0 rpy=3.14159 0.0 1.57
- joint laser_left_joint: origin xyz=0.22 0.14 0.01 rpy=1.2024826  -0.39149955  2.20542129 -> xyz=0.15 0.14 0.01 rpy=1.2024826  -0.39149955  2.20542129
- joint laser_right_joint: origin xyz=0.21 -0.16 0.01 rpy=-1.190795   -0.44884566 -2.31588007 -> xyz=0.15 -0.8 0.01 rpy=-1.190795   -0.44884566 -2.31588007
- joint velodyne_joint: origin xyz=0.085 0.0 0.035 rpy=0.0 0.07574228249456938 0.0 -> xyz=0.0 0.0 0.05 rpy=0.0 0.0 0.0

Commit message: still tuning..

File: cartographer_ros/urdf/m6_cky.urdf (robot description, URDF)
Before this commit: robot cartographer_backpack_3d, 5 links, 4 joints
Joints:
- joint laser_left_joint: origin xyz=0.15 0.14 0.01 rpy=1.2024826  -0.39149955  2.20542129 -> xyz=0.15 0.09 -0.05 rpy=-0.94156  -0.950657  -3.1303
- joint laser_right_joint: origin xyz=0.15 -0.8 0.01 rpy=-1.190795   -0.44884566 -2.31588007 -> xyz=0.15 -0.09 -0.05 rpy=0.94156   -0.950657 3.1303
