Commit message: m6 online and offline test

File: cartographer_ros/urdf/m6.urdf (robot description, URDF)
Before this commit: robot cartographer_backpack_2d, 5 links, 4 joints
Links:
- removed link laser_left
- removed link laser_right
Joints:
- removed joint laser_left_link_joint
- removed joint laser_right_link_joint
- joint imu_link_joint: origin xyz=0 0 0 rpy=3.141592653 0.0 0.0 -> xyz=0 0 0 rpy=0.0 0.0 0.0

File: cartographer_ros/urdf/m6_yd.urdf (robot description, URDF)
Before this commit: robot cartographer_backpack_2d, 4 links, 3 joints
Links:
- removed link aft_mapped
- added link laser_left; visual cylinder length=0.07 radius=0.05
- added link laser_right; visual cylinder length=0.07 radius=0.05
- link velodyne: geometry visual cylinder length=0.07 radius=0.05
Joints:
- removed joint camera_to_base
- removed joint horizontal_laser_link_joint
- added joint laser_left_joint: type fixed, parent velodyne, child laser_left, origin xyz=0.12 0.09 -0.12 rpy=1.21044  -0.245674  2.18578
- added joint laser_right_joint: type fixed, parent velodyne, child laser_right, origin xyz=0.12 -0.09 -0.12 rpy=1.93115  -2.89592 0.955809
- added joint velodyne_joint: type fixed, parent base_link, child velodyne, origin xyz=0.13 0.0 0.05 rpy=0.0 0.0 0.0
- joint imu_link_joint: origin xyz=0 0 0 rpy=3.14159 0.0 1.57 -> xyz=0.0 0.0 0.0 rpy=3.14159 0.0 1.57

File: cartographer_ros/urdf/m6_yq.urdf (robot description, URDF)
Before this commit: robot cartographer_backpack_2d, 4 links, 3 joints
Links:
- removed link aft_mapped
- link velodyne: geometry visual cylinder length=0.07 radius=0.05
Joints:
- removed joint camera_to_base
- removed joint horizontal_laser_link_joint
- added joint velodyne_joint: type fixed, parent base_link, child velodyne, origin xyz=0.0 0.0 0.05 rpy=0.0 0.0 0.0
- joint imu_link_joint: origin xyz=0 0 0 rpy=3.14159 0.0 1.57 -> xyz=0.0 0.0 0.0 rpy=3.14159 0.0 1.57

File: cartographer_ros/urdf/yida_2d.urdf (robot description, URDF)
Before this commit: robot cartographer_backpack_2d, 4 links, 3 joints
Links:
- removed link aft_mapped
Joints:
- removed joint camera_to_base
- removed joint horizontal_laser_link_joint
- added joint velodyne_joint: type fixed, parent base_link, child velodyne, origin xyz=0.0 0.0 0.05 rpy=0.0 0.0 0.0
- joint imu_link_joint: origin xyz=0 0 0 rpy=3.14159 0.0 1.57 -> xyz=0.0 0.0 0.0 rpy=3.14159 0.0 1.57
